File: pca20065/pca20065.kicad_pcb (KiCad board)
At the start: 6 copper layers, 53 x 53 mm, 243 parts, among them J1 MM8130-2600, J2 MM8130-2600, J3 HDR-3, 1mm, J4 SF72S006VBxR2500, J6 USB-C 2.0, M1 nRF9151-LACAA1A, P1 HDR-4, 1mm, P8 Pin Header 2x5, P9 Card Edge, 0.8mm, Q1 RV2C010UNT2L, Q13 DMC2990UDJ, Q14 RV2C010UNT2L, Q2 DMN2990UDJ, Q3 RV2C010UNT2L, Q4 DMN2990UDJ, Q6 DMC2990UDJ, SW1 Switch, SW2 AYZ0102AGRLC, SW3 PB SW, SW4 L-KLS7-TS5401A-1.35-250-T, U1 NLAS5223BMNR2G, U11 nPM1300-QEAAC0, U12 FSA2466UMX, U13 TCK106AG, U14 TCK106AG, U15 MFFx_M2M_UICC, U16 NX3DV2567, U17 QM13345, U18 BMI270, U20 ADXL367, U23 BME688, U24 TXS0102YZPR, U26 BMM350, U3 TCK106AG, U4 TCK106AG, U7 GD25LE255ELIG, U8 ECMF02-4CMX8, U9 SKY65943-11, X1 32MHz, X2 32.768kHz

Commit message: Cleaned up
Parts:
- removed C55: 100nF, pca20065-import-fps:CAPC0603X03L_C
- removed P8: Pin Header 2x5, pca20065-import-fps:HDR_2x5-SMD-1.27mm-ANG
- removed P9: Card Edge, 0.8mm, pca20065-import-fps:10056847-101LF
- removed R17: 10k, pca20065-import-fps:RESC0603X03L_C
- removed R18: 100k, pca20065-import-fps:RESC0603X03L_C
- removed R32: 0R, pca20065-import-fps:RESC0603X03L_C
- removed SW1: Switch, pca20065-import-fps:JS102011JAQN
- removed SW2: AYZ0102AGRLC, pca20065-import-fps:AYZ0102AGRLC
- removed TP27, TP28, TP29: Ø1.5mm,SMD, pca20065-import-fps:TP_SMD_D1.5mm
- removed U1: NLAS5223BMNR2G, pca20065-import-fps:UFQFN40P140X180X55-10N
- removed U12: FSA2466UMX, pca20065-import-fps:XQFN40P180X260X50-16N
Connections:
- M1 pad 5: /Interface/TRACE.CLK -> (no net)
Routing:
- net 1V8_SW: track 163.1 -> 130.5 mm, vias 39 -> 34
- net /Interface/FSA_COM.CH1: track 22.0 -> 0.00 mm, vias 4 -> 0
- net /Interface/FSA_COM.CH2: track 20.9 -> 0.00 mm, vias 4 -> 0
- net /Interface/FSA_NO.CH1: track 18.7 -> 0.00 mm, vias 4 -> 0
- net /Interface/RESET: track 17.3 -> 0.00 mm, vias 4 -> 0
- net /Interface/TRACE.TRACE1: track 14.5 -> 0.25 mm, vias 5 -> 1
- net /Interface/nRF54_SWD.RST: track 28.6 -> 15.6 mm, vias 8 -> 6
- net /Interface/TRACE.CLK: track 9.42 -> 0.00 mm, vias 5 -> 0
- net /Interface/Switch_FSA/IN 1-2: track 7.16 -> 0.00 mm, vias 5 -> 0
- net /Interface/TRACE.TRACE0: track 37.9 -> 32.0 mm, vias 7 -> 5
- net /Interface/FSA_NO.CH3: track 5.83 -> 0.00 mm, vias 1 -> 0
- net VDD_nRF91_RES: track 5.68 -> 0.00 mm
- net 1V8: track 29.9 -> 25.0 mm, vias 4 -> 3
- net VSYS: track 23.2 -> 18.9 mm, vias 4 -> 2
- net /Interface/EXP_BOARD.PIN1: track 37.8 -> 34.0 mm, vias 5 -> 4
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