File: pca20065/pca20065_nrf54l15.kicad_sch (KiCad schematic)
At the start: 26 parts, among them U6 nRF54L15-QFAA, X1 ${ALTIUM_VALUE}, X2 ${ALTIUM_VALUE}

Commit message: Cleaned up
Parts:
- added J7: TC2030-NL, pca20065-import-fps:Tag-Connect_TC2030-IDC-NL_2x03_P1.27mm_Vertical, symbol pca20065:TC2030_SWD_UART
Connections:
- net GND: now also J7.5 (GND)
- net VDD_nRF54: now also J7.1 (VCC)
- net nRF54_SWD.CLK: now also J7.4 (SWDCLK)
- net nRF54_SWD.IO: now also J7.2 (SWDIO)
- net nRF91_SWD.IO: now reaches U6.14 (P2.03)
- net nRF91_SWD.CLK: now reaches U6.17 (P2.06/TRACECLK)
- net nRF91_SWD.RST: now reaches U6.21 (P2.10/TRACEDATA(3))
- net DBG_TX: now reaches U6.3 (P1.02/NFC1)
- net DBG_TX: now also J7.6 (TX)
- net DBG_RX: now reaches U6.4 (P1.03/NFC2)
- net DBG_RX: now also J7.3 (RX)
- no-connect marks 5 -> 0
Other:
- note added: "J7: nRF54L15 SWD + debug UART (P1.02 TX, P1.03 RX)"
- note added: "P2.03/P2.06/P2.10: SWD master to nRF9151 (flash nRF91 from nRF54)"
