File: pca20065/pca20065_nrf9151.kicad_sch (KiCad schematic)
At the start: 33 parts, among them M1 ${ALTIUM_VALUE}, Q13 ${ALTIUM_VALUE}, Q14 ${ALTIUM_VALUE}, U9 ${ALTIUM_VALUE}

Commit message: Replaced nrf5340 with nrf54l15
Connections:
- net WIFI_HOST_IF.ENABLE: no longer names the net of M1.47 (P0.28)
- net WIFI_HOST_IF.IRQ: no longer names the net of M1.77 (P0.16)
- net WIFI_HOST_IF.SS: no longer names the net of M1.78 (P0.17)
- net WIFI_HOST_IF.VDDIO_CTRL: no longer names the net of M1.45 (P0.27)
- net nRF53_SWD.RST renamed nRF54_SWD.RST
- no-connect marks 23 -> 22
Other:
- note added: "nRF54_RESET"
- note removed: "WIFI_SS"
- note removed: "nRF53_RESET"

Commit message: Cleaned up
Parts:
- added J8: TC2030-NL, pca20065-import-fps:Tag-Connect_TC2030-IDC-NL_2x03_P1.27mm_Vertical, symbol pca20065:TC2030_SWD_UART
Connections:
- net 1V8_SW: now also J8.1 (VCC)
- net GND: now also J8.5 (GND)
- net nRF91_SWD.CLK: now also J8.4 (SWDCLK)
- net nRF91_SWD.IO: now also J8.2 (SWDIO)
- net DBG_TX: now reaches M1.77 (P0.16)
- net DBG_TX: now also J8.6 (TX)
- net DBG_RX: now reaches M1.78 (P0.17)
- net DBG_RX: now also J8.3 (RX)
- net TRACE.CLK: no longer names the net of M1.5 (P0.21)
- no-connect marks 22 -> 21
Other:
- note added: "J8: nRF9151 SWD + debug UART (P0.16 TX, P0.17 RX)"
- note removed: "BUCKEN"
- note removed: "HOST_IRQ"
- note removed: "VDDIO_CTRL"
