File: pca20065/pca20065_power_supply.kicad_sch (KiCad schematic)
At the start: 75 parts, among them J3 ${ALTIUM_VALUE}, SW1 ${ALTIUM_VALUE}, U11 ${ALTIUM_VALUE}, U13 ${ALTIUM_VALUE}, U14 ${ALTIUM_VALUE}, U2 ${ALTIUM_VALUE}, U25 ${ALTIUM_VALUE}, U3 ${ALTIUM_VALUE}, U4 ${ALTIUM_VALUE}, U5 ${ALTIUM_VALUE}

Commit message: Replaced nrf5340 with nrf54l15
Parts:
- removed C77: ${ALTIUM_VALUE}, pca20065-import-fps:CAPC1608X06L, symbol pca20065:CAP_8
- removed C78: ${ALTIUM_VALUE}, pca20065-import-fps:CAPC1608X06L, symbol pca20065:CAP_6
- removed C80: ${ALTIUM_VALUE}, pca20065-import-fps:CAPC1608X06L, symbol pca20065:CAP_9
- removed C81: ${ALTIUM_VALUE}, pca20065-import-fps:CAPC1608X06L, symbol pca20065:CAP_7
- removed C82, C83, C84, C85: ${ALTIUM_VALUE}, pca20065-import-fps:CAPC0603X03L_C, symbol pca20065:CAP
- removed L10: ${ALTIUM_VALUE}, pca20065-import-fps:INDC1608X06L, symbol pca20065:IND_1
- removed L9: ${ALTIUM_VALUE}, pca20065-import-fps:INDC2016X10N, symbol pca20065:IND
- removed R25: ${ALTIUM_VALUE}, pca20065-import-fps:RESC0603X03L_C_NC, symbol pca20065:RES_1
- removed R9: ${ALTIUM_VALUE}, pca20065-import-fps:RESC0603X03L_C, symbol pca20065:RES
- removed TP11: ${ALTIUM_VALUE}, pca20065-import-fps:TP_SMD_D1.0mm, symbol pca20065:TESTPAD_2
- removed TP13, TP14: ${ALTIUM_VALUE}, pca20065-import-fps:TP_SMD_D1.5mm, symbol pca20065:TESTPAD
- removed U2: ${ALTIUM_VALUE}, pca20065-import-fps:BGA4C40P2X2_76X76X62, symbol pca20065:TCK106AG
- removed U25: ${ALTIUM_VALUE}, pca20065-import-fps:BGA45C40P5X9_217X364X49, symbol pca20065:nPM6001_CAAA
- removed U5: ${ALTIUM_VALUE}, pca20065-import-fps:BGA4C40P2X2_76X76X62, symbol pca20065:TCK108AG
Connections:
- net RFFE_BLE_WIFI_ENABLE: no longer names the net of U11.8 (GPIO1)
- net VDD_nRF53 renamed VDD_nRF54
- net nPM60_ENABLE: no longer names the net of U11.29 (LSOUT1/VOUTLDO1)
- net nPM60_READY: no longer names the net of U11.11 (GPIO4)
- no-connect marks 11 -> 12
Other:
- note removed: "I2C address: 0x70"
- note removed: "nRF7002 PMIC"

Commit message: Cleaned up
Parts:
- removed SW1: ${ALTIUM_VALUE}, pca20065-import-fps:JS102011JAQN, symbol pca20065:SW-DPDT
- added ST10, ST11: Net tie, pca20065-import-fps:NetTie-2_SMD_Pad2.0mm, symbol pca20065:2 pin starpoint
Connections:
- net 1V8: now also ST10.1
- net 1V8_SW: now also ST10.2
- net VSYS: now also ST11.1
- net VSYS_SW: now also ST11.2
Other:
- note added: "Battery connector"
- note added: "SW1 removed: always on (off = nPM1300 ship mode)"
- note removed: "Battery connector and power switch"
